Commit message: current working project

File: robots/simple.urdf (robot description, URDF)
Before this commit: robot humanoid_robot, 5 links, 4 joints
Links:
- removed link left_arm_link1
- removed link left_arm_link2
- removed link right_arm_link1
- removed link right_arm_link2
- added link left_hand, mass 0.1; collision box size=0.3 0.05 0.3; visual box size=0.3 0.05 0.3
- added link left_leg, mass 1; collision cylinder length=0.4 radius=0.05; visual cylinder length=0.4 radius=0.05
- added link left_lower_arm, mass 0.8; collision cylinder length=0.5 radius=0.03; visual cylinder length=0.5 radius=0.03
- added link left_upper_arm, mass 1.5; collision cylinder length=0.8 radius=0.04; visual cylinder length=0.8 radius=0.04
- added link right_hand, mass 0.1; collision box size=0.3 0.05 0.3; visual box size=0.3 0.05 0.3
- added link right_leg, mass 1; collision cylinder length=0.4 radius=0.05; visual cylinder length=0.4 radius=0.05
- added link right_lower_arm, mass 0.8; collision cylinder length=0.5 radius=0.03; visual cylinder length=0.5 radius=0.03
- added link right_upper_arm, mass 1.5; collision cylinder length=0.8 radius=0.04; visual cylinder length=0.8 radius=0.04
- link base_link: geometry collision capsule length=0.9 radius=0.25; visual capsule length=0.9 radius=0.25
Joints:
- added joint left_hand_joint: type fixed, parent left_lower_arm, child left_hand, origin xyz=0 0 0.5 rpy=0 0 0
- added joint left_leg_joint: type fixed, parent base_link, child left_leg, origin xyz=0.12 0 -0.2 rpy=0 0 0
- added joint right_hand_joint: type fixed, parent right_lower_arm, child right_hand, origin xyz=0 0 0.5 rpy=0 1.5708 0
- added joint right_leg_joint: type fixed, parent base_link, child right_leg, origin xyz=-0.12 0 -0.2 rpy=0 0 0
- joint left_elbow: child left_arm_link2 -> left_lower_arm; limit lower=-2.0944 upper=0 effort=20 velocity=10 -> lower=-2.09 upper=2.09 effort=60 velocity=2.0; origin xyz=0 0 0.4 rpy=0 0 0 -> xyz=0 0 0.6 rpy=0 0 0; parent left_arm_link1 -> left_upper_arm
- joint left_shoulder: child left_arm_link1 -> left_upper_arm; limit lower=-1.5708 upper=1.5708 effort=20 velocity=10 -> lower=-3.14 upper=3.14 effort=100 velocity=2.0; origin xyz=0.15 0 0.7 rpy=0 0 0 -> xyz=0.3 0 0.7 rpy=0 0 0
- joint right_elbow: child right_arm_link2 -> right_lower_arm; limit lower=-2.0944 upper=0 effort=20 velocity=10 -> lower=-2.09 upper=2.09 effort=60 velocity=2.0; origin xyz=0 0 0.4 rpy=0 0 0 -> xyz=0 0 0.6 rpy=0 0 0; parent right_arm_link1 -> right_upper_arm
- joint right_shoulder: child right_arm_link1 -> right_upper_arm; limit lower=-1.5708 upper=1.5708 effort=20 velocity=10 -> lower=-3.14 upper=3.14 effort=100 velocity=2.0; origin xyz=-0.15 0 0.7 rpy=0 0 0 -> xyz=-0.3 0 0.7 rpy=0 0 0
